File: Lab10/Lab10/pt_2.kicad_sch (KiCad schematic)
At the start: 8 parts, among them Q1 IRF9540N, Q2 2N4401-AP

Commit message: update sch
Parts:
- added Q3: 2N4403-AP, digikey-footprints:TO-92-3_Formed_Leads, symbol dk_Transistors-Bipolar-BJT-Single:2N4403-AP
- added U10: L293D, digikey-footprints:DIP-16_W7.62mm, symbol dk_PMIC-Motor-Drivers-Controllers:L293D
- R1: value 4.7k -> 10
- R2: value 4.7k -> 10k
Connections:
- net +12V: now also Q3.3 (C); no longer Q2.1 (E)
- net VCC: now also Q2.3 (C); no longer R1.1
- net at Q2.2 (B), R2.2: now also Q3.2 (B)
- net at Q1.1 (G), R1.2: no longer Q2.3 (C)
- new net: Q2.1 (E), Q3.1 (E), R1.1
