File: Lab10/Lab10/_autosave-pt_1.kicad_sch (KiCad schematic)
At the start: 15 parts, among them U4 LM339, U5 LM324, U6 uA7812

Commit message: SCH done
Parts:
- removed C3: 10n, symbol Device:C
- removed R10, R11, R15, R17, R18, R19: 10k, symbol Device:R
- removed R12, R14: 1.8k, symbol Device:R
- removed R13, R16: 1k, symbol Device:R
- removed RV2: 100k, symbol Device:R_Potentiometer
- removed U4: LM339, symbol Comparator:LM339
- removed U5: LM324, symbol Amplifier_Operational:LM324
- removed U6: uA7812, symbol Regulator_Linear:uA7812
- added C2: 10n, symbol Device:C
- added R3, R4, R6: 10k, symbol Device:R
- added R5: 4.7k, symbol Device:R
- added R7, R9: 1.8k, symbol Device:R
- added R8: 1k, symbol Device:R
- added RV1: 100k, symbol Device:R_Potentiometer
- added U1: LM324, symbol Amplifier_Operational:LM324
- added U2: uA7812, symbol Regulator_Linear:uA7812
- added U3: LM339, symbol Comparator:LM339
Connections:
- net +12V: now also R6.1, RV1.1, U1.4 (V+), U2.3 (OUT)
- net GND: now also R3.2, R4.2, U1.11 (V-), U2.2 (GND), U3.12 (V-)
- net PWM: now also R5.2, U3.2
- net TRI: now also C2.2, R8.1, U1.1, U3.4 (-)
- net VCC: now also R5.1, U2.1 (IN), U3.3 (V+)
- new net: C2.1, R7.2, U1.2 (-)
- new net: R8.2, R9.1, U1.5 (+)
- new net: R4.1, R6.2, U1.3 (+), U1.6 (-)
- new net: R7.1, R9.2, U1.7
- new net: R3.1, RV1.2, U3.5 (+)
Other:
- note added: "Lm339 Vmax is 30V so we can run it off Vcc and so PWM voltage=VCC"
