File: Lab10/Lab10/_autosave-pt_2.kicad_sch (KiCad schematic)
At the start: 8 parts, among them Q1 IRF9540N, Q2 2N4401-AP

Commit message: SCH done
Parts:
- R2: value 4.7k -> 10k
Changed lines of the file:
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@@
 			)
 		)
-		(property "Value" "4.7k"
+		(property "Value" "10k"
 			(at 111.76 113.03 90)
 			(effects
