File: Lab10/Lab10/pt5.kicad_sch (KiCad schematic)
At the start: 0 parts

Commit message: SCH done
Parts:
- added C4: 10n, symbol Device:C
- added R20, R21, R25, R26, R27, R28: 10k, symbol Device:R
- added R22, R24: 1.8k, symbol Device:R
- added R23, R29: 1k, symbol Device:R
- added RV3: 100k, symbol Device:R_Potentiometer
- added U7: LM339, symbol Comparator:LM339
- added U8: LM324, symbol Amplifier_Operational:LM324
- added U9: uA7812, symbol Regulator_Linear:uA7812
Connections:
- new net: C4.1, R22.2, U8.2 (-)
- new net: R20.2, R21.1, U8.3 (+), U8.6 (-)
- new net: R25.1, RV3.2, U8.10 (+)
- new net: R23.2, R24.1, U8.5 (+)
- new net: R28.1, U7.5 (+), U8.8
- new net: R22.1, R24.2, U8.7
- new net: R26.1, U8.9 (-)
- new net +12V: R20.1, R29.1, RV3.1, U7.3 (V+), U8.4 (V+), U9.3 (OUT)
- new net GND: R21.2, R25.2, R27.2, R28.2, U7.12 (V-), U8.11 (V-), U9.2 (GND)
- new net PWM: R29.2, U7.1, U7.2
- new net TRI: C4.2, R23.1, U7.4 (-), U8.1
- new net VCC: U9.1 (IN)
- new net VDC: R26.2, R27.1
Other:
- note added: "1/(2RC) = 27.7Khz"
- note added: "12V linear reg"
- note added: "Error amplifier"
- note added: "PWM Generator"
- note added: "Set reference voltage to set PWM duty cycle"
- note added: "Triangle wave osc"
- note added: "comperater and shunt for current limit"
- note added: "offset for osc"
