File: Lab10/Lab10/pt_1.kicad_sch (KiCad schematic)
At the start: 3 parts, among them U1 LM324, U2 uA7812, U3 LM339

Commit message: Changes
Parts:
- added C2: 10n, symbol Device:C
- added R3, R4, R6: 10k, symbol Device:R
- added R5: 1k, symbol Device:R
- added RV1: 100k, symbol Device:R_Potentiometer
- added unit 3 of U1
- added unit 2 of U3
Connections:
- net GND: now also R3.2, R4.2
- net at U1.6 (-): now also U1.3 (+), R4.1, R6.2
- net +12V: now reaches U3.3 (V+)
- net +12V: now also U1.4 (V+), U2.3 (OUT), R5.1, R6.1, RV1.1
- net at U1.1: now also U3.4 (-), C2.2
- net at U1.2 (-): now also C2.1
- net PWM: now reaches U3.2
- net PWM: now also R5.2
- net at U3.5 (+): now also R3.1, RV1.2
- net VCC: now reaches U2.1 (IN)
Other:
- note added: "12V linear reg"
- note added: "Error amplifier"
- note added: "Set reference voltage to set PWM duty cycle"
- note added: "comperater and shunt for current limit"
- note added: "offset for osc"
- moved on the sheet: U1A

Commit message: SCH done
Parts:
- added R7, R9: 1.8k, symbol Device:R
- added R8: 1k, symbol Device:R
- added U10: L7809, symbol Regulator_Linear:L7809
Connections:
- net +12V: now also U10.3 (OUT)
- net GND: now also U10.2 (GND)
- net VCC: now also U10.1 (IN)
- net at C2.1, U1.2 (-): now also R7.2
- net TRI: now reaches C2.2, U1.1, U3.4 (-)
- net TRI: now also R8.1
- net at U1.5 (+): now also R8.2, R9.1
- net at U1.7: now also R7.1, R9.2
Other:
- note added: "1/(2RC) = 27.7Khz"
- note added: "9V linear reg"
- note added: "Triangle wave osc"
- moved on the sheet: U1C, U3B

Commit message: update sch
Parts:
- removed R7, R9: 1.8k, symbol Device:R
- removed R8: 1k, symbol Device:R
- removed unit 2 of U1
- removed unit 1 of U1
- removed U10: L7809, symbol Regulator_Linear:L7809
- added C6: 10n, symbol Device:C
- added R30: 470k, symbol Device:R
- added U11: NE555D, Package_SO:SOIC-8_3.9x4.9mm_P1.27mm, symbol Timer:NE555D
- C2: value 10n -> 4.7n
- R4: value 10k -> 1.8k
- R5: value 1k -> 1.8k
- R6: value 10k -> 4.7k
Connections:
- net +12V: now also R4.1, U11.4 (R), U11.8 (VCC); no longer R5.1, R6.1, U3.3 (V+)
- net GND: now also C2.2, C6.2, U11.1 (GND); no longer R4.2
- net PWM: now also R30.2
- net TRI: now also U11.3 (Q); no longer C2.2
- net VCC: now also R5.1, U3.3 (V+)
- net at C2.1: now also R6.2, U11.2 (TR), U11.6 (THR)
- net at R3.1, RV1.2, U3.5 (+): now also R30.1
- new net: R4.2, R6.1, U11.7 (DIS)
- new net: C6.1, U11.5 (CV)
Other:
- note added: "Aprox: Triangle Wave (RC value from 555)"
- note added: "Lm339 Vmax is 30V so we can run it off Vcc and so PWM voltage=VCC"
- note added: "hysterious resistor"
- note removed: "1/(2RC) = 27.7Khz"
- note removed: "9V linear reg"
- note removed: "Triangle wave osc"
- note removed: "offset for osc"
