File: Lab10/Lab10/_autosave-pt3.kicad_sch (KiCad schematic)
At the start: 15 parts, among them U7 LM339, U8 LM324, U9 uA7812

Commit message: 3ab11
Parts:
- removed C4: 10n, symbol Device:C
- removed R20, R21, R25, R26, R27, R28: 10k, symbol Device:R
- removed R22, R24: 1.8k, symbol Device:R
- removed R23, R29: 1k, symbol Device:R
- removed RV3: 100k, symbol Device:R_Potentiometer
- removed U7: LM339, symbol Comparator:LM339
- removed U8: LM324, symbol Amplifier_Operational:LM324
- removed U9: uA7812, symbol Regulator_Linear:uA7812
- added C3: 10n, symbol Device:C
- added C7: 100n, symbol Device:C
- added R10, R11, R17, R18, R19: 10k, symbol Device:R
- added R12, R14: 1.8k, symbol Device:R
- added R13, R16: 1k, symbol Device:R
- added RV2: 100k, symbol Device:R_Potentiometer
- added U1, U5: LM324, symbol Amplifier_Operational:LM324
- added U4: LM339, symbol Comparator:LM339
- added U6: uA7812, symbol Regulator_Linear:uA7812
Connections:
- net +12V: now also R10.1, R16.1, RV2.1, U4.3 (V+), U5.4 (V+), U6.3 (OUT)
- net GND: now also R11.2, R18.2, R19.2, U4.12 (V-), U5.11 (V-), U6.2 (GND)
- net PWM: now also R16.2, U4.2
- net TRI: now also C3.2, R13.1, U4.4 (-)
- net VCC: now also U6.1 (IN)
- net VDC: now also R17.2, R18.1
- new net: R12.1, R14.2, U5.7
- new net: C3.1, R12.2
- new net: R13.2, R14.1, U5.5 (+)
- new net: C7.1, R19.1, RV2.2, U1.2 (-)
- new net: R10.2, R11.1, U5.6 (-)
- new net: C7.2, U1.1, U4.5 (+)
- new net: R17.1, U1.3 (+)
