File: Lab10/Lab10/pt3.kicad_sch (KiCad schematic)
At the start: 15 parts, among them U4 LM339, U5 LM324, U6 uA7812

Commit message: 3ab11
Parts:
- removed R15: 10k, symbol Device:R
- removed unit 3 of U5
- removed unit 1 of U5
- added U1: LM324, symbol Amplifier_Operational:LM324
Connections:
- net at R19.1, RV2.2: now also U4.5 (+), U1.1, U1.2 (-)
- net at R17.1: now also U1.3 (+)

Commit message: Lab 11
Parts:
- added C7: 100n, symbol Device:C
- added unit 2 of U1
Connections:
- net at R19.1, RV2.2, U1.2 (-): now also C7.1; no longer U1.1, U4.5 (+)
- new net: C7.2, U1.1, U4.5 (+)
Other:
- moved on the sheet: U4B
