File: Lab 11/lab11_motorControl/Pt1_PWM.kicad_sch (KiCad schematic)
At the start: 10 parts, among them U1 NE555D, U2 LM339

Commit message: Lab 11
Parts:
- added unit 5 of U2
- added U3: uA7812, symbol Regulator_Linear:uA7812
- added U4: LM324, symbol Amplifier_Operational:LM324
- C2: value 4.7n -> 10n
Connections:
- net +12V: now also U3.3 (OUT)
- net GND: now also U2.12 (V-), U3.2 (GND)
- net TRI: now also C2.1, R2.2, U1.2 (TR), U1.6 (THR); no longer U1.3 (Q)
- net VCC: now also U2.3 (V+), U3.1 (IN)
Other:
- note added: "12V linear reg"

Commit message: lab 11
Parts:
- removed unit 2 of U4
- added C3: 100n, symbol Device:C
- added R8: 68k, symbol Device:R
- added R9: 100k, symbol Device:R
- added unit 5 of U4
Connections:
- net GND: now also C3.2, R9.2; no longer C2.2
- net at R4.1, U2.5 (+): now also R8.2, R9.1; no longer R3.1, RV1.2
- net at U4.1: now also U4.2 (-), R8.1
- net at U4.3 (+): now also R3.1, RV1.2
- new net: C2.2, C3.1
Other:
- moved on the sheet: U4A

Commit message: Lab 11
Parts:
- removed R8: 68k, symbol Device:R
- removed R9: 100k, symbol Device:R
- removed unit 1 of U4
Connections:
- net at R4.1, U2.5 (+): now also R3.1, RV1.2
