File: Lab 11/lab11_motorControl/Pt2.kicad_sch (KiCad schematic)
At the start: 0 parts

Commit message: Lab 11
Parts:
- added D1: D_Schottky, symbol Device:D_Schottky
- added M1: Motor_DC, symbol Motor:Motor_DC
- added Q1: 2N4401-AP, digikey-footprints:TO-92-3_Formed_Leads, symbol dk_Transistors-Bipolar-BJT-Single:2N4401-AP
- added Q2: 2N4403-AP, digikey-footprints:TO-92-3_Formed_Leads, symbol dk_Transistors-Bipolar-BJT-Single:2N4403-AP
- added Q3: IRF540N, Package_TO_SOT_THT:TO-220-3_Vertical, symbol Transistor_FET:IRF540N
- added R6: 1k, symbol Device:R
- added R7: 10, symbol Device:R
Connections:
- new net: Q1.1 (E), Q2.1 (E), R7.1
- new net: Q1.2 (B), Q2.2 (B), R6.2
- new net: D1.1 (K), M1.1 (+)
- new net: D1.2 (A), M1.2 (-), Q3.2 (D)
- new net: Q3.1 (G), R7.2
- new net +12V: Q1.3 (C)
- new net GND: Q2.3 (C)
- new net PWM: R6.1
Other:
- note added: "Vcc can vary between 16 and 28V Vgs (max) is 20V so don't pull gate low to turn on Pull to 12V that always hit our -4V (max) threshold voltage"

Commit message: Lab 11
Connections:
- net GND: now also Q3.3 (S)
Changed lines of the file:
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@@
+		)
+	)
+	(symbol
+		(lib_id "power:GND")
+		(at 161.29 107.95 0)
+		(unit 1)
+		(exclude_from_sim no)
+		(in_bom yes)
+		(on_board yes)
+		(dnp no)
+		(fields_autoplaced yes)
+		(property "Reference" "#PWR018"
+			(at 161.29 114.3 0)
+			(effects
+				(font
+					(size 1.27 1.27)
+				)
+				(hide yes)
+			)
+		)
+		(property "Value" "GND"
+			(at 161.29 113.03 0)
+			(effects
+				(font
+					(size 1.27 1.27)
+				)
+			)
+		)
+		(property "Footprint" ""
+			(at 161.29 107.95 0)
+			(effects
+				(font
+					(size 1.27 1.27)
+				)
+				(hide yes)
+			)
+		)
+		(property "Datasheet" ""
+			(at 161.29 107.95 0)
+			(effects
+				(font
+					(size 1.27 1.27)
+				)
+				(hide yes)
+			)
+		)
+		(property "Description" "Power symbol creates a global label with name \"GND\" , ground"
+			(at 161.29 107.95 0)
+			(effects
+				(font
+					(size 1.27 1.27)
+				)
+				(hide yes)
+			)
+		)
+		(pin "1"
+		)
+		(instances
+			(project "lab11_motorControl"
+				(path "/a010efed-9821-4af0-b24d-85bee303b04d/cfe5cd27-5e6e-40e6-9097-28550d4f32b7"
+					(reference "#PWR018")
+					(unit 1)
+				)
+			)
 		)
 	)
