File: Lab 11/lab11_motorControl/Sheetname Pt6_ClosingTheLoop.kicad_sch (KiCad schematic)
At the start: 0 parts

Commit message: lab 11
Parts:
- added U4: LM324, symbol Amplifier_Operational:LM324
Changed lines of the file:
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@@
 	(generator_version "8.0")
 	(paper "A4")
+	(symbol
+		(lib_id "Amplifier_Operational:LM324")
+		(at 132.08 116.84 0)
+		(unit 2)
+		(exclude_from_sim no)
+		(in_bom yes)
+		(on_board yes)
+		(dnp no)
+		(fields_autoplaced yes)
+		(property "Reference" "U4"
+			(at 132.08 106.68 0)
+			(effects
+				(font
+					(size 1.27 1.27)
+				)
+			)
+		)
+		(property "Value" "LM324"
+			(at 132.08 109.22 0)
+			(effects
+				(font
+					(size 1.27 1.27)
+				)
+			)
+		)
+		(property "Footprint" ""
+			(at 130.81 114.3 0)
+			(effects
+				(font
+					(size 1.27 1.27)
+				)
+				(hide yes)
+			)
+		)
+		(property "Datasheet" "http://www.ti.com/lit/ds/symlink/lm2902-n.pdf"
+			(at 133.35 111.76 0)
+			(effects
+				(font
+					(size 1.27 1.27)
+				)
+				(hide yes)
+			)
+		)
+		(property "Description" "Low-Power, Quad-Operational Amplifiers, DIP-14/SOIC-14/SSOP-14"
+			(at 132.08 116.84 0)
+			(effects
+				(font
+					(size 1.27 1.27)
+				)
+				(hide yes)
+			)
+		)
+		(pin "4"
+		)
+		(pin "7"
+		)
+		(pin "14"
+		)
+		(pin "2"
+		)
+		(pin "6"
+		)
+		(pin "12"
+		)
+		(pin "10"
+		)
+		(pin "11"
+		)
+		(pin "3"
+		)
+		(pin "9"
+		)
+		(pin "13"
+		)
+		(pin "5"
+		)
+		(pin "8"
+		)
+		(pin "1"
+		)
+		(instances
+			(project "lab11_motorControl"
+				(path "/a010efed-9821-4af0-b24d-85bee303b04d/95ef5eee-833e-4c89-8ba9-1d8bf97897bd"
+					(reference "U4")
+					(unit 2)
+				)
+			)
+		)
+	)
 )

Commit message: Lab 11
Parts:
- removed U4: LM324, symbol Amplifier_Operational:LM324
- added C10: 2.2u, symbol Device:C
- added C11: 100n, symbol Device:C
- added C9: 10u, symbol Device:C
- added R21: 33k, symbol Device:R
- added R22, R9: 10k, symbol Device:R
- added R23: 0, symbol Device:R
- added R24: 470k, symbol Device:R
- added R25: 1.8k, symbol Device:R
- added R8: 820k, symbol Device:R
- added RV2: 100k, symbol Device:R_Potentiometer
- added U4: LM324, symbol Amplifier_Operational:LM324
- added U5: LM339, symbol Comparator:LM339
Connections:
- new net: C10.2, C11.2, C9.2, R24.1, U4.1, U5.5 (+)
- new net: R9.1, RV2.2, U4.3 (+)
- new net: R21.1, R22.1, R23.1, R8.2, U4.2 (-)
- new net: C11.1, R23.2
- new net: C10.1, R22.2
- new net: C9.1, R21.2
- new net +12V: RV2.1
- new net GND: R9.2
- new net PWM: R24.2, R25.2, U5.2
- new net TRI: U5.4 (-)
- new net VCC: R25.1
- new net Voltage_RPM: R8.1
Other:
- note added: "Vref"
- note added: "hysterious resistor"
