File: Lab 11/lab11_motorControl/lab11_motorControl.kicad_sch (KiCad schematic)
At the start: 0 parts

Commit message: Lab 11
Other:
- added sheet Pt6_ClosingTheLoop (Sheetname Pt6_ClosingTheLoop.kicad_sch)
- added sheet V_FrequencyToVoltage (PartV.kicad_sch)
Changed lines of the file:
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@@
+	)
+	(sheet
+		(at 121.92 97.79)
+		(size 26.67 19.05)
+		(fields_autoplaced yes)
+		(stroke
+			(width 0.1524)
+			(type solid)
+		)
+		(fill
+			(color 0 0 0 0.0000)
+		)
+		(property "Sheetname" "Pt6_ClosingTheLoop"
+			(at 121.92 97.0784 0)
+			(effects
+				(font
+					(size 1.27 1.27)
+				)
+				(justify left bottom)
+			)
+		)
+		(property "Sheetfile" "Sheetname Pt6_ClosingTheLoop.kicad_sch"
+			(at 121.92 117.4246 0)
+			(effects
+				(font
+					(size 1.27 1.27)
+				)
+				(justify left top)
+			)
+		)
+		(instances
+			(project "lab11_motorControl"
+				(path "/a010efed-9821-4af0-b24d-85bee303b04d"
+					(page "5")
+				)
+			)
+		)
+	)
+	(sheet
+		(at 87.63 93.98)
+		(size 22.86 21.59)
+		(fields_autoplaced yes)
+		(stroke
+			(width 0.1524)
+			(type solid)
+		)
+		(fill
+			(color 0 0 0 0.0000)
+		)
+		(property "Sheetname" "V_FrequencyToVoltage"
+			(at 87.63 93.2684 0)
+			(effects
+				(font
+					(size 1.27 1.27)
+				)
+				(justify left bottom)
+			)
+		)
+		(property "Sheetfile" "PartV.kicad_sch"
+			(at 87.63 116.1546 0)
+			(effects
+				(font
+					(size 1.27 1.27)
+				)
+				(justify left top)
+			)
+		)
+		(instances
+			(project "lab11_motorControl"
+				(path "/a010efed-9821-4af0-b24d-85bee303b04d"
+					(page "4")
+				)
+			)
+		)
 	)
 	(sheet

Commit message: Lab 11
Other:
- added sheet SampleAndHold (untitled.kicad_sch)
Changed lines of the file:
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@@
+		)
+	)
+	(sheet
+		(at 184.15 90.17)
+		(size 25.4 27.94)
+		(fields_autoplaced yes)
+		(stroke
+			(width 0.1524)
+			(type solid)
+		)
+		(fill
+			(color 0 0 0 0.0000)
+		)
+		(property "Sheetname" "SampleAndHold"
+			(at 184.15 89.4584 0)
+			(effects
+				(font
+					(size 1.27 1.27)
+				)
+				(justify left bottom)
+			)
+		)
+		(property "Sheetfile" "untitled.kicad_sch"
+			(at 184.15 118.6946 0)
+			(effects
+				(font
+					(size 1.27 1.27)
+				)
+				(justify left top)
+			)
+		)
+		(instances
+			(project "lab11_motorControl"
+				(path "/a010efed-9821-4af0-b24d-85bee303b04d"
+					(page "6")
+				)
+			)
 		)
 	)
