File: lab12/lab12/Laser_signal.kicad_sch (KiCad schematic)
At the start: 44 parts, among them U1 MC7805CT-BP, U10 LM324, U14 LM324, U2 NE555D, U5 LM324, U8 LM339

Commit message: adding values
Parts:
- C6: value C -> 2.2u
- C7: value C -> 200p
- R16, R22, R23, R24: value R -> 10k
- R17: value R -> 560k
Connections:
- net +5V: now also R14.1, RV1.1, RV2.1
- net GND: now also R21.1, R22.2, R3.2
Other:
- moved on the sheet: C6, R17

Commit message: clean up sch
Parts:
- added R34, R36: 10k, symbol Device:R
- added R35: 56k, symbol Device:R
- added RV4: R_Potentiometer, symbol Device:R_Potentiometer
- R16: value 10k -> 100k
- R18, R20, R6: value R -> 10k
- R19: value R -> 0
- R21, R4, R5: value R -> 56k
Connections:
- net GND: now also R35.1
- net Voltage_Solar: now also R34.1; no longer D2.1 (K), U10.5 (+)
- net at U8.7 (+): now also R36.1, RV4.2
- net at C7.2: now also D2.1 (K), U10.5 (+), R34.2, R35.2
Other:
- note added: "set vref for center"
- note added: "set vref so diff is min at center"

Commit message: Code for lab 13
Other:
- company: (none) -> CWRU
- moved on the sheet: C1, C2, C3, C4, C5, C6, C7, D2, LD1, R1, R10, R11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
