File: lab12/lab12/StateLogic.kicad_sch (KiCad schematic)
At the start: 8 parts, among them Q1 2N4403-AP, Q5 2N4403-AP, Q6 2N4403-AP, Q7 2N4403-AP, U12 LM339, U9 4011

Commit message: adding values
Parts:
- added R29, R30, R31, R32: R, symbol Device:R
- added R33: 1M, symbol Device:R
- added RV3: R_Potentiometer, symbol Device:R_Potentiometer
- R25, R26: value R -> 1k
Connections:
- net at U12.5 (+): now also R31.2, R32.1
- net at U12.7 (+): now also R29.2, R30.1
- new net: R33.1, RV3.2
- new net GND: R30.2, R32.2, R33.2
Other:
- moved on the sheet: R25, R26, U9E

Commit message: clean up sch
Parts:
- added Q8: 2N4403-AP, digikey-footprints:TO-92-3_Formed_Leads, symbol dk_Transistors-Bipolar-BJT-Single:2N4403-AP
- added Q9: 2N4401-AP, digikey-footprints:TO-92-3_Formed_Leads, symbol dk_Transistors-Bipolar-BJT-Single:2N4401-AP
- added R37, R38: R, symbol Device:R
- added R41, R42: 1k, symbol Device:R
Connections:
- net +5V: now also Q6.1 (E), Q7.1 (E), R29.1, R31.1, RV3.1, Q8.1 (E)
- net GND: now also Q9.1 (E)
- net at R26.2, U12.2, U9.6: now also Q6.2 (B), Q9.2 (B), R38.2
- net at R31.2, R32.1, U12.5 (+): now also R38.1
- net at R25.2, U12.1, U9.1: now also Q7.2 (B), Q8.2 (B), R37.2
- net at Q5.3 (C): now also R42.1
- net at Q1.3 (C): now also R41.1
- net at U12.4 (-): now also R33.1, RV3.2, U12.6 (-)
- net PWM: now reaches Q6.3 (C)
- net PWM: now also Q8.3 (C)
- net at R29.2, R30.1, U12.7 (+): now also R37.1
- net DIR: now reaches Q7.3 (C)
- net DIR: now also Q9.3 (C)
- new net JogLeft: R41.2
- new net JogRight: R42.2
Other:
- note added: "Limits"
- note added: "Seek"
- moved on the sheet: Q1, Q5, Q6, Q7, R25, R26, R29, R30, R31, R32, R33, RV3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

Commit message: Code for lab 13
Other:
- company: (none) -> CWRU
Changed lines of the file:
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@@
 	(generator_version "8.0")
 	(paper "A4")
+	(title_block
+		(company "CWRU")
+		(comment 1 "Drawn by: Toby Cowles")
+	)
 	(junction
 		(at 73.66 124.46)
