File: lab12/lab12/lab12.kicad_sch (KiCad schematic)
At the start: 0 parts

Commit message: clean up sch
Other:
- note added: "ECSE 471 Lab 12: Laser Tracker"
- note removed: "Lab 12: Laser Tracker"
Changed lines of the file:
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@@
 	(generator_version "8.0")
 	(paper "A4")
-	(text "Lab 12: Laser Tracker"
+	(text "ECSE 471\nLab 12: Laser Tracker"
 		(exclude_from_sim no)
-		(at 141.478 48.768 0)
+		(at 164.338 77.978 0)
 		(effects
 			(font
@@
 	(symbol
 		(lib_id "Graphic:SYM_LASER_Large")
-		(at 45.72 48.26 0)
+		(at 99.06 68.58 0)
 		(unit 1)
 		(exclude_from_sim yes)
@@
 		(fields_autoplaced yes)
 		(property "Reference" "#SYM1"
-			(at 45.72 43.18 0)
+			(at 99.06 63.5 0)
 			(effects
 				(font
@@
 		)
 		(property "Value" "SYM_LASER_Large"
-			(at 45.72 54.991 0)
+			(at 99.06 75.311 0)
 			(effects
 				(font
@@
 		)
 		(property "Footprint" ""
-			(at 45.466 52.705 0)
+			(at 98.806 73.025 0)
 			(effects
 				(font
@@
 		)
 		(property "Datasheet" "~"
-			(at 46.482 53.34 0)
+			(at 99.822 73.66 0)
 			(effects
 				(font
@@
 		)
 		(property "Description" "Laser radiation warning symbol, large"
-			(at 45.72 48.26 0)
+			(at 99.06 68.58 0)
 			(effects
 				(font
@@
 	)
 	(sheet
-		(at 171.45 97.79)
+		(at 149.86 101.6)
 		(size 29.21 20.32)
 		(fields_autoplaced yes)
@@
 		)
 		(property "Sheetname" "StateLogic"
-			(at 171.45 97.0784 0)
+			(at 149.86 100.8884 0)
 			(effects
 				(font
@@
 		)
 		(property "Sheetfile" "StateLogic.kicad_sch"
-			(at 171.45 118.6946 0)
+			(at 149.86 122.5046 0)
 			(effects
 				(font
@@
 	)
 	(sheet
-		(at 67.31 92.71)
+		(at 63.5 100.33)
 		(size 29.21 21.59)
 		(fields_autoplaced yes)
@@
 		)
 		(property "Sheetname" "MotorControl"
-			(at 67.31 91.9984 0)
+			(at 63.5 99.6184 0)
 			(effects
 				(font
@@
 		)
 		(property "Sheetfile" "motor.kicad_sch"
-			(at 67.31 114.8846 0)
+			(at 63.5 122.5046 0)
 			(effects
 				(font
@@
 	)
 	(sheet
-		(at 77.47 138.43)
+		(at 201.93 95.25)
 		(size 24.13 25.4)
 		(fields_autoplaced yes)
@@
 		)
 		(property "Sheetname" "jog"
-			(at 77.47 137.7184 0)
+			(at 201.93 94.5384 0)
 			(effects
 				(font
@@
 		)
 		(property "Sheetfile" "untitled.kicad_sch"
-			(at 77.47 164.4146 0)
+			(at 201.93 121.2346 0)
 			(effects
 				(font
@@
 	)
 	(sheet
-		(at 110.49 90.17)
+		(at 106.68 97.79)
 		(size 25.4 25.4)
 		(fields_autoplaced yes)
@@
 		)
 		(property "Sheetname" "Laser_signal"
-			(at 110.49 89.4584 0)
+			(at 106.68 97.0784 0)
 			(effects
 				(font
@@
 		)
 		(property "Sheetfile" "Laser_signal.kicad_sch"
-			(at 110.49 116.1546 0)
-			(effects
-				(font
+			(at 106.68 123.7746 0)
+			(effects
+				(font

Commit message: Code for lab 13
Other:
- company: (none) -> CWRU
Changed lines of the file:
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@@
 	(generator_version "8.0")
 	(paper "A4")
+	(title_block
+		(company "CWRU")
+		(comment 1 "Drawn by: Toby Cowles")
+	)
 	(text "ECSE 471\nLab 12: Laser Tracker"
 		(exclude_from_sim no)
