File: lab12/lab12/motor.kicad_sch (KiCad schematic)
At the start: 5 parts, among them M1 Motor_DC, U3 L293D, U4 40106, U6 LM339, U7 CD4066BE

Commit message: clean up sch
Other:
- moved on the sheet: U4C
Changed lines of the file:
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@@
 	(symbol
 		(lib_id "4xxx:40106")
-		(at 242.57 80.01 0)
+		(at 45.72 109.22 0)
 		(unit 3)
 		(exclude_from_sim no)
@@
 		(fields_autoplaced yes)
 		(property "Reference" "U4"
-			(at 242.57 71.12 0)
+			(at 45.72 100.33 0)
 			(effects
 				(font
@@
 		)
 		(property "Value" "40106"
-			(at 242.57 73.66 0)
+			(at 45.72 102.87 0)
 			(effects
 				(font
@@
 		)
 		(property "Footprint" ""
-			(at 242.57 80.01 0)
+			(at 45.72 109.22 0)
 			(effects
 				(font
@@
 		)
 		(property "Datasheet" "https://assets.nexperia.com/documents/data-sheet/HEF40106B.pdf"
-			(at 242.57 80.01 0)
+			(at 45.72 109.22 0)
 			(effects
 				(font
@@
 		)
 		(property "Description" "Hex Schmitt trigger inverter"
-			(at 242.57 80.01 0)
+			(at 45.72 109.22 0)
 			(effects
 				(font

Commit message: Code for lab 13
Other:
- company: (none) -> CWRU
Changed lines of the file:
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@@
 	(generator_version "8.0")
 	(paper "A4")
+	(title_block
+		(company "CWRU")
+		(comment 1 "Drawn by: Toby Cowles")
+	)
 	(junction
 		(at 203.2 121.92)
