File: lab12/lab12/untitled.kicad_sch (KiCad schematic)
At the start: 6 parts, among them Q2 2N4403-AP, Q3 2N4401-AP, Q4 2N4403-AP, SW1 SW_Push, SW2 SW_Push, U11 40106

Commit message: clean up sch
Parts:
- added R39, R40: 10k, symbol Device:R
Connections:
- net GND: now also R39.2, R40.2
- net JogLeft: now also R39.1
- net JogRight: now also R40.1
Other:
- moved on the sheet: Q2, Q3, Q4, SW1, SW2, U11A, U11B, U11C, U11G

Commit message: Code for lab 13
Other:
- company: (none) -> CWRU
Changed lines of the file:
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@@
 	(generator_version "8.0")
 	(paper "A4")
+	(title_block
+		(company "CWRU")
+		(comment 1 "Drawn by: Toby Cowles")
+	)
 	(junction
 		(at 99.06 115.57)
