File: lab13/Lab13_Sch/lab13/Digital.kicad_sch (KiCad schematic)
At the start: 5 parts, among them SW1 SW_Push, U2 RP2040, U3 4N35

Commit message: Finish lab13 start lab 14
Parts:
- added BZ1: Buzzer, symbol Device:Buzzer
- added R10: 220, symbol Device:R
- added U6: MAN71A, Display_7Segment:MAN71A, symbol Display_Character:MAN71A
- C3: value C -> 1n
Connections:
- net +5V: now also R10.2
- net GND: now also BZ1.2 (-)
- net at U2.11 (GPIO8): now also U6.8 (D)
- net at U2.12 (GPIO9): now also U6.7 (E)
- net at U2.13 (GPIO10): now also U6.2 (F)
- net at U2.14 (GPIO11): now also U6.11 (G)
- net at U2.27 (GPIO16): now also BZ1.1 (+)
- net at U2.7 (GPIO5): now also U6.1 (A)
- net at U2.8 (GPIO6): now also U6.13 (B)
- net at U2.9 (GPIO7): now also U6.10 (C)
- new net: R10.1, U6.14 (CA), U6.3 (CA)
Other:
- note added: "Drive buzzer with 4khz tone"
- company: (none) -> CWRU
- title: (none) -> Lab 13: Digital Heating Pad Control
- moved on the sheet: U3
