File: lab13/Lab13_Sch/lab13/TRIAC_Drive.kicad_sch (KiCad schematic)
At the start: 11 parts, among them Q2 2N4401-AP, Q4 BT139-600, U5 4N35

Commit message: Finish lab13 start lab 14
Parts:
- added C6: 10n, symbol Device:C
- added LA1: Lamp, symbol Device:Lamp
- added R8: 1k, symbol Device:R
- added R9: 220, symbol Device:R
Connections:
- net 30v: now also Q4.2 (A2), C6.1; no longer R7.1
- net AC_N: now also LA1.1 (-), R8.2
- net TRIAC: now reaches U5.1
- net at U5.2: now also R9.1
- net at C5.2, D8.2 (A), Q2.1 (E): now also R7.2; no longer U5.4
- net at Q2.3 (C), R6.1: now also U5.5
- net at Q4.1 (A1): now also LA1.2 (+)
- new net: Q2.2 (B), R7.1, U5.4
- new net: C6.2, R8.1
- new net GND: R9.2
Other:
- company: (none) -> CWRU
- title: (none) -> Lab 13: Digital Heating Pad Control
- moved on the sheet: Q2, Q4, R6, U5
