File: lab13/Lab13_Sch/lab13/lab13.kicad_sch (KiCad schematic)
At the start: 4 parts, among them Q1 2N4401-AP, Q3 BT139-600, U1 MOC3020M

Commit message: Finish lab13 start lab 14
Parts:
- removed D1: D, symbol Device:D
- removed Q1: 2N4401-AP, digikey-footprints:TO-92-3_Formed_Leads, symbol dk_Transistors-Bipolar-BJT-Single:2N4401-AP
- removed Q3: BT139-600, Package_TO_SOT_THT:TO-220-3_Vertical, symbol Triac_Thyristor:BT139-600
- removed U1: MOC3020M, symbol Relay_SolidState:MOC3020M
Other:
- note added: "ECSE 471 Lab 13: Digital Heating Pad Control"
- company: (none) -> CWRU
- title: (none) -> Lab 13: Digital Heating Pad Control
