File: Lab14/lab14_distance_sensor/Transmitter.kicad_sch (KiCad schematic)
At the start: 4 parts, among them U1 NE555P, U2 NE555P, U3 NE555P

Commit message: work on lab 14
Parts:
- added C1, C2: 10n, symbol Device:C
- added R1: 1.8k, symbol Device:R
- added R2: 180, symbol Device:R
Connections:
- net GND: now reaches U3.1 (GND)
- net GND: now also LS1.2, U2.1 (GND), C1.2, C2.2
- net at U3.2 (TR): now also U3.6 (THR), C1.1, R1.2
- net at U3.3 (Q): now also LS1.1
- net at U3.4 (R): now also U2.3 (Q)
- net at U3.5 (CV): now also C2.1
- net at U3.7 (DIS): now also R1.1, R2.2
- net Transmitting: now reaches U1.3 (Q)
- net at U2.2 (TR): now also U2.6 (THR)
Other:
- moved on the sheet: LS1, U3

Commit message: more work on lab 14
Other:
- company: (none) -> CWRU
- title: (none) -> ECSE 471 Lab 14
Changed lines of the file:
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@@
 	(generator_version "8.0")
 	(paper "A4")
+	(title_block
+		(title "ECSE 471 Lab 14")
+		(date "2025-04-24")
+		(company "CWRU")
+		(comment 1 "Drawn By T.Cowles")
+	)
 	(junction
 		(at 261.62 116.84)

Commit message: lab 14
Parts:
- removed U2: NE555P, Package_DIP:DIP-8_W7.62mm, symbol Timer:NE555P
- added C5, C6: 10n, symbol Device:C
- added C7: 2.2u, symbol Device:C
- added R6: 330k, symbol Device:R
- added R7: 500 ohm pot, symbol Device:R
- added U6: 40106, symbol 4xxx:40106
Connections:
- net GND: now also C5.2, C6.2, C7.2
- net at U1.2 (TR): now also U1.6 (THR), C7.1, R7.2
- net at U1.4 (R): now also U1.8 (VCC)
- net at U1.5 (CV): now also C5.1
- net at U1.7 (DIS): now also R6.2, R7.1
- net at U3.4 (R): now also U6.2
- net Transmitting renamed !Transmitting
- net !Transmitting: now also U6.1
- new net: C6.1, U6.14 (VDD)
Other:
- note removed: "50% duty cycle: few hundred hertz for pulses"
- moved on the sheet: U1
