File: Lab14/lab14_distance_sensor/memory.kicad_sch (KiCad schematic)
At the start: 0 parts

Commit message: work on lab 14
Parts:
- added C3: 10u, symbol Device:C
- added SW1: SW_Push, symbol Switch:SW_Push
- added U4: LM324, symbol Amplifier_Operational:LM324
Connections:
- new net: C3.1, SW1.2
- new net GND: C3.2

Commit message: more work on lab 14
Parts:
- added BZ1: Buzzer, symbol Device:Buzzer
- added unit 3 of U4
Other:
- company: (none) -> CWRU
- title: (none) -> ECSE 471 Lab 14
Changed lines of the file:
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@@
 	(generator_version "8.0")
 	(paper "A4")
+	(title_block
+		(title "ECSE 471 Lab 14")
+		(date "2025-04-24")
+		(company "CWRU")
+		(comment 1 "Drawn By T.Cowles")
+	)
 	(wire
 		(pts
@@
 			(width 0)
 			(type default)
+		)
+	)
+	(symbol
+		(lib_id "Device:Buzzer")
+		(at 194.31 86.36 0)
+		(unit 1)
+		(exclude_from_sim no)
+		(in_bom yes)
+		(on_board yes)
+		(dnp no)
+		(fields_autoplaced yes)
+		(property "Reference" "BZ1"
+			(at 198.12 85.0899 0)
+			(effects
+				(font
+					(size 1.27 1.27)
+				)
+				(justify left)
+			)
+		)
+		(property "Value" "Buzzer"
+			(at 198.12 87.6299 0)
+			(effects
+				(font
+					(size 1.27 1.27)
+				)
+				(justify left)
+			)
+		)
+		(property "Footprint" ""
+			(at 193.675 83.82 90)
+			(effects
+				(font
+					(size 1.27 1.27)
+				)
+				(hide yes)
+			)
+		)
+		(property "Datasheet" "~"
+			(at 193.675 83.82 90)
+			(effects
+				(font
+					(size 1.27 1.27)
+				)
+				(hide yes)
+			)
+		)
+		(property "Description" "Buzzer, polarized"
+			(at 194.31 86.36 0)
+			(effects
+				(font
+					(size 1.27 1.27)
+				)
+				(hide yes)
+			)
+		)
+		(pin "1"
+		)
+		(pin "2"
+		)
+		(instances
+			(project "lab14_distance_sensor"
+				(path "/dc193204-f06f-4bda-a794-1fc81970e56e/63fcc152-d205-4771-b903-c6ac1fa49597"
+					(reference "BZ1")
+					(unit 1)
+				)
+			)
 		)
 	)
@@
 				)
 			)
+		)
+	)
+	(symbol
+		(lib_id "Amplifier_Operational:LM324")
+		(at 119.38 124.46 0)
+		(unit 3)
+		(exclude_from_sim no)
+		(in_bom yes)
+		(on_board yes)
+		(dnp no)
+		(fields_autoplaced yes)
+		(property "Reference" "U4"
+			(at 119.38 114.3 0)
+			(effects
+				(font
+					(size 1.27 1.27)
+				)
+			)
+		)
+		(property "Value" "LM324"
+			(at 119.38 116.84 0)
+			(effects
+				(font
+					(size 1.27 1.27)
+				)
+			)
+		)
+		(property "Footprint" ""
+			(at 118.11 121.92 0)
+			(effects
+				(font
+					(size 1.27 1.27)
+				)
+				(hide yes)
+			)
+		)
+		(property "Datasheet" "http://www.ti.com/lit/ds/symlink/lm2902-n.pdf"
+			(at 120.65 119.38 0)
+			(effects
+				(font
+					(size 1.27 1.27)
+				)
+				(hide yes)
+			)
+		)
+		(property "Description" "Low-Power, Quad-Operational Amplifiers, DIP-14/SOIC-14/SSOP-14"
+			(at 119.38 124.46 0)
+			(effects
+				(font
+					(size 1.27 1.27)
+				)
+				(hide yes)
+			)
+		)
+		(pin "8"
+		)
+		(pin "14"
+		)
+		(pin "11"
+		)
+		(pin "13"
+		)
+		(pin "2"
+		)
+		(pin "7"
+		)
+		(pin "5"
+		)
+		(pin "6"
+		)
+		(pin "10"
+		)
+		(pin "1"
+		)
+		(pin "9"
+		)
+		(pin "4"
+		)
+		(pin "12"
+		)
+		(pin "3"
+		)
+		(instances
+			(project "lab14_distance_sensor"
+				(path "/dc193204-f06f-4bda-a794-1fc81970e56e/63fcc152-d205-4771-b903-c6ac1fa49597"
+					(reference "U4")
+					(unit 3)
+				)
+			)

Commit message: lab 14
Parts:
- removed U4: LM324, symbol Amplifier_Operational:LM324
Changed lines of the file:
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@@
-	)
-	(symbol
-		(lib_id "Amplifier_Operational:LM324")
-		(at 124.46 76.2 0)
-		(unit 4)
-		(exclude_from_sim no)
-		(in_bom yes)
-		(on_board yes)
-		(dnp no)
-		(fields_autoplaced yes)
-		(property "Reference" "U4"
-			(at 124.46 66.04 0)
-			(effects
-				(font
-					(size 1.27 1.27)
-				)
-			)
-		)
-		(property "Value" "LM324"
-			(at 124.46 68.58 0)
-			(effects
-				(font
-					(size 1.27 1.27)
-				)
-			)
-		)
-		(property "Footprint" ""
-			(at 123.19 73.66 0)
-			(effects
-				(font
-					(size 1.27 1.27)
-				)
-				(hide yes)
-			)
-		)
-		(property "Datasheet" "http://www.ti.com/lit/ds/symlink/lm2902-n.pdf"
-			(at 125.73 71.12 0)
-			(effects
-				(font
-					(size 1.27 1.27)
-				)
-				(hide yes)
-			)
-		)
-		(property "Description" "Low-Power, Quad-Operational Amplifiers, DIP-14/SOIC-14/SSOP-14"
-			(at 124.46 76.2 0)
-			(effects
-				(font
-					(size 1.27 1.27)
-				)
-				(hide yes)
-			)
-		)
-		(pin "8"
-		)
-		(pin "14"
-		)
-		(pin "11"
-		)
-		(pin "13"
-		)
-		(pin "2"
-		)
-		(pin "7"
-		)
-		(pin "5"
-		)
-		(pin "6"
-		)
-		(pin "10"
-		)
-		(pin "1"
-		)
-		(pin "9"
-		)
-		(pin "4"
-		)
-		(pin "12"
-		)
-		(pin "3"
-		)
-		(instances
-			(project "lab14_distance_sensor"
-				(path "/dc193204-f06f-4bda-a794-1fc81970e56e/63fcc152-d205-4771-b903-c6ac1fa49597"
-					(reference "U4")
-					(unit 4)
-				)
-			)
-		)
 	)
 	(symbol
@@
 				)
 			)
-		)
-	)
-	(symbol
-		(lib_id "Amplifier_Operational:LM324")
-		(at 119.38 124.46 0)
-		(unit 3)
-		(exclude_from_sim no)
-		(in_bom yes)
-		(on_board yes)
-		(dnp no)
-		(fields_autoplaced yes)
-		(property "Reference" "U4"
-			(at 119.38 114.3 0)
-			(effects
-				(font
-					(size 1.27 1.27)
-				)
-			)
-		)
-		(property "Value" "LM324"
-			(at 119.38 116.84 0)
-			(effects
-				(font
-					(size 1.27 1.27)
-				)
-			)
-		)
-		(property "Footprint" ""
-			(at 118.11 121.92 0)
-			(effects
-				(font
-					(size 1.27 1.27)
-				)
-				(hide yes)
-			)
-		)
-		(property "Datasheet" "http://www.ti.com/lit/ds/symlink/lm2902-n.pdf"
-			(at 120.65 119.38 0)
-			(effects
-				(font
-					(size 1.27 1.27)
-				)
-				(hide yes)
-			)
-		)
-		(property "Description" "Low-Power, Quad-Operational Amplifiers, DIP-14/SOIC-14/SSOP-14"
-			(at 119.38 124.46 0)
-			(effects
-				(font
-					(size 1.27 1.27)
-				)
-				(hide yes)
-			)
-		)
-		(pin "8"
-		)
-		(pin "14"
-		)
-		(pin "11"
-		)
-		(pin "13"
-		)
-		(pin "2"
-		)
-		(pin "7"
-		)
-		(pin "5"
-		)
-		(pin "6"
-		)
-		(pin "10"
-		)
-		(pin "1"
-		)
-		(pin "9"
-		)
-		(pin "4"
-		)
-		(pin "12"
-		)
-		(pin "3"
-		)
-		(instances
-			(project "lab14_distance_sensor"
-				(path "/dc193204-f06f-4bda-a794-1fc81970e56e/63fcc152-d205-4771-b903-c6ac1fa49597"
-					(reference "U4")
-					(unit 3)
-				)
-			)
