File: Lab14/lab14_distance_sensor/receiver.kicad_sch (KiCad schematic)
At the start: 0 parts

Commit message: work on lab 14
Parts:
- added D1, D2: D, symbol Device:D
- added Q1: 2N4401-AP, digikey-footprints:TO-92-3_Formed_Leads, symbol dk_Transistors-Bipolar-BJT-Single:2N4401-AP
- added R3: R, symbol Device:R
- added U4: LM324, symbol Amplifier_Operational:LM324
Connections:
- new net: D1.2 (A), D2.1 (K)
- new net: D2.2 (A), Q1.2 (B), R3.1
- new net: D1.1 (K), Q1.1 (E)

Commit message: more work on lab 14
Parts:
- removed unit 3 of U4
- added C4: C, symbol Device:C
- added U5: CD4066BE, Package_DIP:DIP-14_W7.62mm, symbol Analog_Switch:CD4066BE
Other:
- company: (none) -> CWRU
- title: (none) -> ECSE 471 Lab 14
- moved on the sheet: D1, D2, Q1, R3, U4A, U4E

Commit message: lab 14
Parts:
- added C10, C11: 22n, symbol Device:C
- added C8: 10n, symbol Device:C
- added C9: 1n, symbol Device:C
- added LS2: Speaker_Crystal, symbol Device:Speaker_Crystal
- added R10, R11, R9: 10k, symbol Device:R
- added R12, R13: 2.2k, symbol Device:R
- added R14, R15: 470, symbol Device:R
- added R4: 180k, symbol Device:R
- added R5: 1k, symbol Device:R
- added R8: 100k, symbol Device:R
- added U2: LM324, symbol Amplifier_Operational:LM324
- added unit 3 of U4
- added U7: LM339, symbol Comparator:LM339
Connections:
- net at U4.1: now also C9.1, R4.2
- net at U4.2 (-): now also R4.1, R5.2
- net at U4.3 (+): now also C8.2, R15.2
- net at U4.5 (+): now also C9.2, R14.2
- net at U4.6 (-): now also R8.1, R9.2
- net at U4.7: now also R10.1, R8.2
- net GND: now reaches U4.11 (V-)
- new net: C8.1, LS2.2
- new net: R12.2, R13.2, U4.9 (-)
- new net: C11.1, R10.2, R11.1
- new net: C10.2, R11.2, U4.10 (+)
- new net: C10.1, R12.1
- new net Receive Voltage: C11.2, R13.1, U4.8
Other:
- moved on the sheet: C4, D1, D2, Q1, R3, U4B, U5A, U5B, U5C, U5D
